File: diyalarmclock.sch (KiCad schematic (older format))
At the start: 4 parts, among them P1 CONN_2, U1 LD1117

Commit message: Basic wiring for MCU and RTC.
Still need to add capacitors to the power inputs.
Parts:
- added IC?: LPC812M-SO-20, symbol LPC812M-SO-20
- added IC?: DS3231M-SO-8, symbol DS3231M-SO-8
Connections:
- net labels added: RESET, SCL, SDA
- wire segments 10 -> 25
Changed lines of the file:
@@
 	1200 1500 1800 1500
 Connection ~ 1800 1500
+$Comp
+L LPC812M-SO-20 IC?
+U 1 1 54F24FD2
+P 3150 3750
+F 0 "IC?" H 2700 4700 60  0000 L CNN
+F 1 "LPC812M-SO-20" H 3600 2800 60  0000 R CNN
+F 2 "" H 3150 3750 60  0000 C CNN
+F 3 "" H 3150 3750 60  0000 C CNN
+	1    3150 3750
+	1    0    0    -1
+$EndComp
+$Comp
+L +3.3V #PWR?
+U 1 1 54F24FFC
+P 2300 2850
+F 0 "#PWR?" H 2300 2810 30  0001 C CNN
+F 1 "+3.3V" H 2300 2960 30  0000 C CNN
+F 2 "" H 2300 2850 60  0000 C CNN
+F 3 "" H 2300 2850 60  0000 C CNN
+	1    2300 2850
+	1    0    0    -1
+$EndComp
+Wire Wire Line
+	2300 2850 2300 3150
+Wire Wire Line
+	2300 2950 2400 2950
+$Comp
+L GND #PWR?
+U 1 1 54F25021
+P 2300 4650
+F 0 "#PWR?" H 2300 4650 30  0001 C CNN
+F 1 "GND" H 2300 4580 30  0001 C CNN
+F 2 "" H 2300 4650 60  0000 C CNN
+F 3 "" H 2300 4650 60  0000 C CNN
+	1    2300 4650
+	1    0    0    -1
+$EndComp
+Wire Wire Line
+	2400 4550 2300 4550
+Wire Wire Line
+	2300 4550 2300 4650
+Wire Wire Line
+	2300 3150 2400 3150
+Connection ~ 2300 2950
+Text GLabel 4000 3850 2    60   Input ~ 0
+SDA
+Text GLabel 4000 3950 2    60   Input ~ 0
+SCL
+Wire Wire Line
+	3900 3850 4000 3850
+Wire Wire Line
+	3900 3950 4000 3950
+$Comp
+L DS3231M-SO-8 IC?
+U 1 1 54F25163
+P 7150 3750
+F 0 "IC?" H 6750 4200 60  0000 L CNN
+F 1 "DS3231M-SO-8" H 7550 3300 60  0000 R CNN
+F 2 "" H 7150 3750 60  0000 C CNN
+F 3 "" H 7150 3750 60  0000 C CNN
+	1    7150 3750
+	1    0    0    -1
+$EndComp
+Text GLabel 7950 3550 2    60   Input ~ 0
+SDA
+Text GLabel 7950 3450 2    60   Input ~ 0
+SCL
+Wire Wire Line
+	7850 3450 7950 3450
+Wire Wire Line
+	7850 3550 7950 3550
+$Comp
+L +3.3V #PWR?
+U 1 1 54F251AD
+P 6350 3350
+F 0 "#PWR?" H 6350 3310 30  0001 C CNN
+F 1 "+3.3V" H 6350 3460 30  0000 C CNN
+F 2 "" H 6350 3350 60  0000 C CNN
+F 3 "" H 6350 3350 60  0000 C CNN
+	1    6350 3350
+	1    0    0    -1
+$EndComp
+Wire Wire Line
+	6350 3350 6350 3450
+Wire Wire Line
+	6350 3450 6450 3450
+$Comp
+L GND #PWR?
+U 1 1 54F251DC
+P 6350 4150
+F 0 "#PWR?" H 6350 4150 30  0001 C CNN
+F 1 "GND" H 6350 4080 30  0001 C CNN
+F 2 "" H 6350 4150 60  0000 C CNN
+F 3 "" H 6350 4150 60  0000 C CNN
+	1    6350 4150
+	1    0    0    -1
+$EndComp
+Wire Wire Line
+	6450 4050 6350 4050
+Wire Wire Line
+	6350 4050 6350 4150
+Text GLabel 4000 2950 2    60   Input ~ 0
+RESET
+Wire Wire Line
+	3900 2950 4000 2950
+Text GLabel 7950 4050 2    60   Input ~ 0
+RESET
+Wire Wire Line
+	7850 4050 7950 4050
 $EndSCHEMATC
