File: mainboard/mainboard.sch (KiCad schematic (older format))
At the start: 25 parts, among them P1 CONN_01X06, P2 CONN_01X08, P3 CONN_01X08, SW1 SW_PUSH, SW2 SW_PUSH, SW3 SW_PUSH, SW4 SW_PUSH, SW5 SW_PUSH, SW6 SW_PUSH, U1 LPC812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

Commit message: Map schematic symbols to footprints.
Parts:
- C1, C2, C4: footprint (none) -> Capacitors_SMD:C_0805_HandSoldering
- C3: footprint (none) -> miniclock:CPOL_SMD_6.3mm
- P1: footprint (none) -> Pin_Headers:Pin_Header_Straight_1x06
- P2, P3: footprint (none) -> Pin_Headers:Pin_Header_Straight_1x08
- R1, R2, R3, R4, R5, R6, R7, R8, R9: footprint (none) -> Resistors_SMD:R_0805_HandSoldering
- SW1, SW2, SW3, SW4, SW5, SW6: footprint (none) -> miniclock:PUSHSWITCH
- U1: footprint (none) -> Housings_SOIC:SOIC-20_7.5x12.8mm_Pitch1.27mm
- U2: footprint (none) -> Housings_SOIC:SOIC-8_3.9x4.9mm_Pitch1.27mm
- VR1: footprint (none) -> miniclock:SOT223
Changed lines of the file:
@@
 LIBS:valves
 LIBS:parts
+LIBS:mainboard-cache
 EELAYER 25 0
 EELAYER END
@@
 F 0 "VR1" H 9600 1050 60  0000 C CNN
 F 1 "LD1117" H 9950 500 60  0000 C CNN
-F 2 "" H 9750 900 60  0000 C CNN
+F 2 "miniclock:SOT223" H 9750 900 60  0001 C CNN
 F 3 "" H 9750 900 60  0000 C CNN
 	1    9750 900
@@
 F 0 "P1" H 1800 1450 50  0000 C CNN
 F 1 "CONN_01X06" V 1900 1100 50  0000 C CNN
-F 2 "" H 1800 1100 60  0000 C CNN
+F 2 "Pin_Headers:Pin_Header_Straight_1x06" H 1800 1100 60  0001 C CNN
 F 3 "" H 1800 1100 60  0000 C CNN
 	1    1800 1100
@@
 F 0 "C2" H 9175 1250 50  0000 L CNN
 F 1 "C" H 9175 1050 50  0000 L CNN
-F 2 "" H 9188 1000 30  0000 C CNN
+F 2 "Capacitors_SMD:C_0805_HandSoldering" H 9188 1000 30  0001 C CNN
 F 3 "" H 9150 1150 60  0000 C CNN
 	1    9150 1150
@@
 F 0 "C3" H 10375 1250 50  0000 L CNN
 F 1 "CP" H 10375 1050 50  0000 L CNN
-F 2 "" H 10388 1000 30  0000 C CNN
+F 2 "miniclock:CPOL_SMD_6.3mm" H 10388 1000 30  0001 C CNN
 F 3 "" H 10350 1150 60  0000 C CNN
 	1    10350 1150
@@
 F 0 "U1" H 1500 3450 60  0000 C CNN
 F 1 "LPC812" H 2200 2200 60  0000 C CNN
-F 2 "" H 1650 3100 60  0000 C CNN
+F 2 "Housings_SOIC:SOIC-20_7.5x12.8mm_Pitch1.27mm" H 1650 3100 60  0001 C CNN
 F 3 "" H 1650 3100 60  0000 C CNN
 	1    1900 2850
@@
 F 0 "U2" H 4700 1800 60  0000 C CNN
 F 1 "DS3231M" H 5150 1200 60  0000 C CNN
-F 2 "" H 4950 1450 60  0000 C CNN
+F 2 "Housings_SOIC:SOIC-8_3.9x4.9mm_Pitch1.27mm" H 4950 1450 60  0001 C CNN
 F 3 "" H 4950 1450 60  0000 C CNN
 	1    5000 1500
@@
 F 0 "C4" H 5075 2250 50  0000 L CNN
 F 1 "C" H 5075 2050 50  0000 L CNN
-F 2 "" H 5088 2000 30  0000 C CNN
+F 2 "Capacitors_SMD:C_0805_HandSoldering" H 5088 2000 30  0001 C CNN
 F 3 "" H 5050 2150 60  0000 C CNN
 	1    5050 2150
@@
 F 0 "R3" V 5680 1100 50  0000 C CNN
 F 1 "R" V 5600 1100 50  0000 C CNN
-F 2 "" V 5530 1100 30  0000 C CNN
+F 2 "Resistors_SMD:R_0805_HandSoldering" V 5530 1100 30  0001 C CNN
 F 3 "" H 5600 1100 30  0000 C CNN
 	1    5600 1100
@@
 F 0 "R4" V 5880 1100 50  0000 C CNN
 F 1 "R" V 5800 1100 50  0000 C CNN
-F 2 "" V 5730 1100 30  0000 C CNN
+F 2 "Resistors_SMD:R_0805_HandSoldering" V 5730 1100 30  0001 C CNN
 F 3 "" H 5800 1100 30  0000 C CNN
 	1    5800 1100
@@
 F 0 "R1" V 4030 1300 50  0000 C CNN
 F 1 "R" V 3950 1300 50  0000 C CNN
-F 2 "" V 3880 1300 30  0000 C CNN
+F 2 "Resistors_SMD:R_0805_HandSoldering" V 3880 1300 30  0001 C CNN
 F 3 "" H 3950 1300 30  0000 C CNN
 	1    3950 1300
@@
 F 0 "C1" H 1925 3900 50  0000 L CNN
 F 1 "C" H 1925 3700 50  0000 L CNN
-F 2 "" H 1938 3650 30  0000 C CNN
+F 2 "Capacitors_SMD:C_0805_HandSoldering" H 1938 3650 30  0001 C CNN
 F 3 "" H 1900 3800 60  0000 C CNN
 	1    1900 3800
@@
 F 0 "P2" H 4650 3950 50  0000 C CNN
 F 1 "CONN_01X08" V 4750 3500 50  0000 C CNN
-F 2 "" H 4650 3500 60  0000 C CNN
+F 2 "Pin_Headers:Pin_Header_Straight_1x08" H 4650 3500 60  0001 C CNN
 F 3 "" H 4650 3500 60  0000 C CNN
 	1    4650 3500
@@
 F 0 "P3" H 5450 3950 50  0000 C CNN
 F 1 "CONN_01X08" V 5550 3500 50  0000 C CNN
-F 2 "" H 5450 3500 60  0000 C CNN
+F 2 "Pin_Headers:Pin_Header_Straight_1x08" H 5450 3500 60  0001 C CNN
 F 3 "" H 5450 3500 60  0000 C CNN
 	1    5450 3500
@@
 F 0 "SW1" H 9800 2810 50  0000 C CNN
 F 1 "SW_PUSH" H 9650 2620 50  0000 C CNN
-F 2 "" H 9650 2700 60  0000 C CNN
+F 2 "miniclock:PUSHSWITCH" H 9650 2700 60  0001 C CNN
 F 3 "" H 9650 2700 60  0000 C CNN
 	1    9650 2700
@@
 F 0 "R2" V 10230 2700 50  0000 C CNN
 F 1 "R" V 10150 2700 50  0000 C CNN
-F 2 "" V 10080 2700 30  0000 C CNN
+F 2 "Resistors_SMD:R_0805_HandSoldering" V 10080 2700 30  0001 C CNN
 F 3 "" H 10150 2700 30  0000 C CNN
 	1    10150 2700
@@
 F 0 "SW2" H 9800 3210 50  0000 C CNN
 F 1 "SW_PUSH" H 9650 3020 50  0000 C CNN
-F 2 "" H 9650 3100 60  0000 C CNN
+F 2 "miniclock:PUSHSWITCH" H 9650 3100 60  0001 C CNN
 F 3 "" H 9650 3100 60  0000 C CNN
 	1    9650 3100
@@
 F 0 "R5" V 10230 3100 50  0000 C CNN
 F 1 "R" V 10150 3100 50  0000 C CNN
-F 2 "" V 10080 3100 30  0000 C CNN
+F 2 "Resistors_SMD:R_0805_HandSoldering" V 10080 3100 30  0001 C CNN
 F 3 "" H 10150 3100 30  0000 C CNN
 	1    10150 3100
@@
 F 0 "SW3" H 9800 3610 50  0000 C CNN
 F 1 "SW_PUSH" H 9650 3420 50  0000 C CNN
-F 2 "" H 9650 3500 60  0000 C CNN
+F 2 "miniclock:PUSHSWITCH" H 9650 3500 60  0001 C CNN
 F 3 "" H 9650 3500 60  0000 C CNN
 	1    9650 3500
@@
 F 0 "R6" V 10230 3500 50  0000 C CNN
 F 1 "R" V 10150 3500 50  0000 C CNN
-F 2 "" V 10080 3500 30  0000 C CNN
+F 2 "Resistors_SMD:R_0805_HandSoldering" V 10080 3500 30  0001 C CNN
 F 3 "" H 10150 3500 30  0000 C CNN
 	1    10150 3500
@@
 F 0 "SW4" H 9800 4010 50  0000 C CNN
 F 1 "SW_PUSH" H 9650 3820 50  0000 C CNN
-F 2 "" H 9650 3900 60  0000 C CNN
+F 2 "miniclock:PUSHSWITCH" H 9650 3900 60  0001 C CNN
 F 3 "" H 9650 3900 60  0000 C CNN
 	1    9650 3900
@@
 F 0 "R7" V 10230 3900 50  0000 C CNN
 F 1 "R" V 10150 3900 50  0000 C CNN
-F 2 "" V 10080 3900 30  0000 C CNN
+F 2 "Resistors_SMD:R_0805_HandSoldering" V 10080 3900 30  0001 C CNN
 F 3 "" H 10150 3900 30  0000 C CNN
 	1    10150 3900
@@
 F 0 "SW5" H 9800 4410 50  0000 C CNN
 F 1 "SW_PUSH" H 9650 4220 50  0000 C CNN
-F 2 "" H 9650 4300 60  0000 C CNN
+F 2 "miniclock:PUSHSWITCH" H 9650 4300 60  0001 C CNN
 F 3 "" H 9650 4300 60  0000 C CNN
 	1    9650 4300
@@
 F 0 "R8" V 10230 4300 50  0000 C CNN
 F 1 "R" V 10150 4300 50  0000 C CNN
-F 2 "" V 10080 4300 30  0000 C CNN
+F 2 "Resistors_SMD:R_0805_HandSoldering" V 10080 4300 30  0001 C CNN
 F 3 "" H 10150 4300 30  0000 C CNN
 	1    10150 4300
@@
 F 0 "SW6" H 9800 4810 50  0000 C CNN
 F 1 "SW_PUSH" H 9650 4620 50  0000 C CNN
-F 2 "" H 9650 4700 60  0000 C CNN
+F 2 "miniclock:PUSHSWITCH" H 9650 4700 60  0001 C CNN
 F 3 "" H 9650 4700 60  0000 C CNN
 	1    9650 4700
@@
 F 0 "R9" V 10230 4700 50  0000 C CNN
 F 1 "R" V 10150 4700 50  0000 C CNN
-F 2 "" V 10080 4700 30  0000 C CNN
+F 2 "Resistors_SMD:R_0805_HandSoldering" V 10080 4700 30  0001 C CNN
 F 3 "" H 10150 4700 30  0000 C CNN
 	1    10150 4700
