File: displayboard/displayboard.sch (KiCad schematic (older format))
At the start: 29 parts, among them P1 CONN_01X08, P2 CONN_01X08, U1 SG-636PCE, U2 LEDM, U3 MAX6960, U4 LEDM, U5 MAX6960, U6 LEDM

Commit message: Assorted updates that I didn't properly distinguish.
Parts:
- removed W1: RED, symbol TEST
- removed W2: BLK, symbol TEST
- removed W3, W6: BLU, symbol TEST
- removed W4, W5: GRN, symbol TEST
- added TP1, TP2, TP3, TP4, TP5, TP6: TESTPOINT, symbol TESTPOINT
- C1, C10, C2, C3, C4, C5, C7, C8, C9, JP1, JP2, JP3, JP4: footprint (none) -> miniclock:0805
- U1: footprint (none) -> miniclock:SG-636PCE
- U2, U4, U6: footprint (none) -> miniclock:KWM-R30881CUYB
- U3, U5: footprint (none) -> miniclock:MAX6960
Connections:
- net +3V3: now also P1.3 (P3), TP2.1 (TP)
- net GND: now also P1.2 (P2), TP1.1 (TP)
- net MISO: now also P1.7 (P7), TP5.1 (TP)
- net MOSI: now also P1.6 (P6), TP4.1 (TP)
- net SCLK: now also P1.5 (P5), TP3.1 (TP)
- net SSEL: now also P1.8 (P8), TP6.1 (TP)
Changed lines of the file:
@@
 Text Notes 5500 7300 0    60   ~ 0
 Mechanical\nconnection\nonly
-Text GLabel 3450 6950 0    60   Output ~ 0
+Text GLabel 3650 6950 0    60   Output ~ 0
 GND
-Text GLabel 3100 7100 0    60   Output ~ 0
+Text GLabel 3650 7050 0    60   Output ~ 0
 +3V3
 Text GLabel 4200 7150 0    60   Output ~ 0
 +3V3
-Text GLabel 3450 7250 0    60   Output ~ 0
+Text GLabel 3650 7250 0    60   Output ~ 0
 SCLK
-Text GLabel 3450 7350 0    60   Output ~ 0
+Text GLabel 3650 7350 0    60   Output ~ 0
 MOSI
-Text GLabel 3450 7450 0    60   Input ~ 0
+Text GLabel 3650 7450 0    60   Input ~ 0
 MISO
-Text GLabel 3450 7550 0    60   Output ~ 0
+Text GLabel 3650 7550 0    60   Output ~ 0
 SSEL
 Text GLabel 4200 6850 0    60   Output ~ 0
 ~RESET
-Wire Wire Line
-	4200 6850 4250 6850
 Wire Wire Line
 	4200 7150 4250 7150
@@
 F 0 "U2" H 9950 1300 60  0000 C CNN
 F 1 "LEDM" H 10900 1300 60  0000 C CNN
-F 2 "" H 10300 1900 60  0000 C CNN
+F 2 "miniclock:KWM-R30881CUYB" H 10300 1900 60  0001 C CNN
 F 3 "" H 10300 1900 60  0000 C CNN
 	1    10450 1900
@@
 F 0 "U4" H 9950 3200 60  0000 C CNN
 F 1 "LEDM" H 10900 3200 60  0000 C CNN
-F 2 "" H 10300 3800 60  0000 C CNN
+F 2 "miniclock:KWM-R30881CUYB" H 10300 3800 60  0001 C CNN
 F 3 "" H 10300 3800 60  0000 C CNN
 	1    10450 3800
@@
 F 0 "U6" H 9950 5100 60  0000 C CNN
 F 1 "LEDM" H 10900 5100 60  0000 C CNN
-F 2 "" H 10300 5700 60  0000 C CNN
+F 2 "miniclock:KWM-R30881CUYB" H 10300 5700 60  0001 C CNN
 F 3 "" H 10300 5700 60  0000 C CNN
 	1    10450 5700
@@
 F 0 "U3" H 1500 3500 60  0000 C CNN
 F 1 "MAX6960" H 2150 600 60  0000 C CNN
-F 2 "" H 1700 1100 60  0000 C CNN
+F 2 "miniclock:MAX6960" H 1700 1100 60  0001 C CNN
 F 3 "" H 1700 1100 60  0000 C CNN
 	1    1900 2100
@@
 F 0 "U5" H 4300 3500 60  0000 C CNN
 F 1 "MAX6960" H 4950 600 60  0000 C CNN
-F 2 "" H 4500 1100 60  0000 C CNN
+F 2 "miniclock:MAX6960" H 4500 1100 60  0001 C CNN
 F 3 "" H 4500 1100 60  0000 C CNN
 	1    4700 2100
@@
 F 0 "JP1" H 1100 2730 50  0000 C CNN
 F 1 "Jumper_NO_Small" H 1110 2590 50  0001 C CNN
-F 2 "" H 1100 2650 60  0000 C CNN
+F 2 "miniclock:0805" H 1100 2650 60  0001 C CNN
 F 3 "" H 1100 2650 60  0000 C CNN
 	1    1100 2650
@@
 F 0 "JP2" H 1100 2830 50  0000 C CNN
 F 1 "Jumper_NO_Small" H 1110 2690 50  0001 C CNN
-F 2 "" H 1100 2750 60  0000 C CNN
+F 2 "miniclock:0805" H 1100 2750 60  0001 C CNN
 F 3 "" H 1100 2750 60  0000 C CNN
 	1    1100 2750
@@
 F 0 "JP3" H 3900 2730 50  0000 C CNN
 F 1 "Jumper_NO_Small" H 3910 2590 50  0001 C CNN
-F 2 "" H 3900 2650 60  0000 C CNN
+F 2 "miniclock:0805" H 3900 2650 60  0001 C CNN
 F 3 "" H 3900 2650 60  0000 C CNN
 	1    3900 2650
@@
 F 0 "JP4" H 3900 2830 50  0000 C CNN
 F 1 "Jumper_NO_Small" H 3910 2690 50  0001 C CNN
-F 2 "" H 3900 2750 60  0000 C CNN
+F 2 "miniclock:0805" H 3900 2750 60  0001 C CNN
 F 3 "" H 3900 2750 60  0000 C CNN
 	1    3900 2750
@@
 F 0 "U1" H 1200 7250 60  0000 C CNN
 F 1 "SG-636PCE" H 1750 6650 60  0000 C CNN
-F 2 "" H 1450 6950 60  0000 C CNN
+F 2 "miniclock:SG-636PCE" H 1450 6950 60  0001 C CNN
 F 3 "" H 1450 6950 60  0000 C CNN
 	1    1450 6950
@@
 F 0 "C1" H 610 7020 50  0000 L CNN
 F 1 "0.1u" H 610 6870 50  0000 L CNN
-F 2 "" H 600 6950 60  0000 C CNN
+F 2 "miniclock:0805" H 600 6950 60  0001 C CNN
 F 3 "" H 600 6950 60  0000 C CNN
 	1    600  6950
@@
 NoConn ~ 5050 7450
 NoConn ~ 5050 7550
-$Comp
-L TEST W2
-U 1 1 565AB0B8
-P 3700 6950
-F 0 "W2" H 3700 6950 40  0000 C CNN
-F 1 "BLK" H 3700 6900 40  0000 C CNN
-F 2 "" H 3700 6950 60  0000 C CNN
-F 3 "" H 3700 6950 60  0000 C CNN
-	1    3700 6950
-	1    0    0    -1
-$EndComp
-$Comp
-L TEST W1
-U 1 1 565AB7DE
-P 3350 7100
-F 0 "W1" H 3350 7100 40  0000 C CNN
-F 1 "RED" H 3350 7050 40  0000 C CNN
-F 2 "" H 3350 7100 60  0000 C CNN
-F 3 "" H 3350 7100 60  0000 C CNN
-	1    3350 7100
-	1    0    0    -1
-$EndComp
-Wire Wire Line
-	3900 6950 4250 6950
-Wire Wire Line
-	3450 6950 3500 6950
-Wire Wire Line
-	3100 7100 3150 7100
-Wire Wire Line
-	3550 7100 3850 7100
-Wire Wire Line
-	3850 7100 3850 7050
-Wire Wire Line
-	3850 7050 4250 7050
-$Comp
-L TEST W3
-U 1 1 565ABE6A
-P 3700 7250
-F 0 "W3" H 3700 7250 40  0000 C CNN
-F 1 "BLU" H 3700 7200 40  0000 C CNN
-F 2 "" H 3700 7250 60  0000 C CNN
-F 3 "" H 3700 7250 60  0000 C CNN
-	1    3700 7250
-	1    0    0    -1
-$EndComp
-$Comp
-L TEST W4
-U 1 1 565ABEC6
-P 3700 7350
-F 0 "W4" H 3700 7350 40  0000 C CNN
-F 1 "GRN" H 3700 7300 40  0000 C CNN
-F 2 "" H 3700 7350 60  0000 C CNN
-F 3 "" H 3700 7350 60  0000 C CNN
-	1    3700 7350
-	1    0    0    -1
-$EndComp
-$Comp
-L TEST W5
-U 1 1 565ABF09
-P 3700 7450
-F 0 "W5" H 3700 7450 40  0000 C CNN
-F 1 "GRN" H 3700 7400 40  0000 C CNN
-F 2 "" H 3700 7450 60  0000 C CNN
-F 3 "" H 3700 7450 60  0000 C CNN
-	1    3700 7450
-	1    0    0    -1
-$EndComp
-$Comp
-L TEST W6
-U 1 1 565ABF53
-P 3700 7550
-F 0 "W6" H 3700 7550 40  0000 C CNN
-F 1 "BLU" H 3700 7500 40  0000 C CNN
-F 2 "" H 3700 7550 60  0000 C CNN
-F 3 "" H 3700 7550 60  0000 C CNN
-	1    3700 7550
-	1    0    0    -1
-$EndComp
-Wire Wire Line
-	3900 7250 4250 7250
-Wire Wire Line
-	3900 7350 4250 7350
-Wire Wire Line
-	3900 7450 4250 7450
-Wire Wire Line
-	3900 7550 4250 7550
 Text Notes 1300 7650 2    60   ~ 0
 Oscillator
@@
 F 0 "C2" H 1310 4520 50  0000 L CNN
 F 1 "0.1u" H 1310 4370 50  0000 L CNN
-F 2 "" H 1300 4450 60  0000 C CNN
+F 2 "miniclock:0805" H 1300 4450 60  0001 C CNN
 F 3 "" H 1300 4450 60  0000 C CNN
 	1    1300 4450
@@
 F 0 "C3" H 1610 4520 50  0000 L CNN
 F 1 "0.1u" H 1610 4370 50  0000 L CNN
-F 2 "" H 1600 4450 60  0000 C CNN
+F 2 "miniclock:0805" H 1600 4450 60  0001 C CNN
 F 3 "" H 1600 4450 60  0000 C CNN
 	1    1600 4450
@@
 F 0 "C4" H 1910 4520 50  0000 L CNN
 F 1 "0.1u" H 1910 4370 50  0000 L CNN
-F 2 "" H 1900 4450 60  0000 C CNN
+F 2 "miniclock:0805" H 1900 4450 60  0001 C CNN
 F 3 "" H 1900 4450 60  0000 C CNN
 	1    1900 4450
@@
 F 0 "C5" H 2210 4520 50  0000 L CNN
 F 1 "0.1u" H 2210 4370 50  0000 L CNN
-F 2 "" H 2200 4450 60  0000 C CNN
+F 2 "miniclock:0805" H 2200 4450 60  0001 C CNN
 F 3 "" H 2200 4450 60  0000 C CNN
 	1    2200 4450
@@
 F 0 "C6" H 2510 4520 50  0000 L CNN
 F 1 "47uF" H 2510 4370 50  0000 L CNN
-F 2 "" H 2500 4450 60  0000 C CNN
+F 2 "" H 2500 4450 60  0001 C CNN
 F 3 "" H 2500 4450 60  0000 C CNN
 	1    2500 4450
@@
 F 0 "C7" H 4110 4520 50  0000 L CNN
 F 1 "0.1u" H 4110 4370 50  0000 L CNN
-F 2 "" H 4100 4450 60  0000 C CNN
+F 2 "miniclock:0805" H 4100 4450 60  0001 C CNN
 F 3 "" H 4100 4450 60  0000 C CNN
 	1    4100 4450
@@
 F 0 "C8" H 4410 4520 50  0000 L CNN
 F 1 "0.1u" H 4410 4370 50  0000 L CNN
-F 2 "" H 4400 4450 60  0000 C CNN
+F 2 "miniclock:0805" H 4400 4450 60  0001 C CNN
 F 3 "" H 4400 4450 60  0000 C CNN
 	1    4400 4450
@@
 F 0 "C9" H 4710 4520 50  0000 L CNN
 F 1 "0.1u" H 4710 4370 50  0000 L CNN
-F 2 "" H 4700 4450 60  0000 C CNN
+F 2 "miniclock:0805" H 4700 4450 60  0001 C CNN
 F 3 "" H 4700 4450 60  0000 C CNN
 	1    4700 4450
@@
 F 0 "C10" H 5010 4520 50  0000 L CNN
 F 1 "0.1u" H 5010 4370 50  0000 L CNN
-F 2 "" H 5000 4450 60  0000 C CNN
+F 2 "miniclock:0805" H 5000 4450 60  0001 C CNN
 F 3 "" H 5000 4450 60  0000 C CNN
 	1    5000 4450
@@
 F 0 "C11" H 5310 4520 50  0000 L CNN
 F 1 "47uF" H 5310 4370 50  0000 L CNN
-F 2 "" H 5300 4450 60  0000 C CNN
+F 2 "" H 5300 4450 60  0001 C CNN
 F 3 "" H 5300 4450 60  0000 C CNN
 	1    5300 4450
@@
 Wire Notes Line
 	5900 5100 5900 600
+Wire Wire Line
+	4250 6850 4200 6850
+$Comp
+L TESTPOINT TP1
+U 1 1 565A7F3D
+P 3750 6950
+F 0 "TP1" H 3750 6900 20  0000 C BNN
+F 1 "TESTPOINT" H 3800 6950 20  0001 L CNN
+F 2 "" H 3750 6950 60  0000 C CNN
+F 3 "" H 3750 6950 60  0000 C CNN
+	1    3750 6950
+	1    0    0    -1
+$EndComp
+$Comp
+L TESTPOINT TP2
+U 1 1 565A81B2
+P 3750 7050
+F 0 "TP2" H 3750 7000 20  0000 C BNN
+F 1 "TESTPOINT" H 3800 7050 20  0001 L CNN
+F 2 "" H 3750 7050 60  0000 C CNN
+F 3 "" H 3750 7050 60  0000 C CNN
+	1    3750 7050
+	1    0    0    -1
+$EndComp
+$Comp
+L TESTPOINT TP3
+U 1 1 565A820D
+P 3750 7250
+F 0 "TP3" H 3750 7200 20  0000 C BNN
+F 1 "TESTPOINT" H 3800 7250 20  0001 L CNN
+F 2 "" H 3750 7250 60  0000 C CNN
+F 3 "" H 3750 7250 60  0000 C CNN
+	1    3750 7250
+	1    0    0    -1
+$EndComp
+$Comp
+L TESTPOINT TP4
+U 1 1 565A8275
+P 3750 7350
+F 0 "TP4" H 3750 7300 20  0000 C BNN
+F 1 "TESTPOINT" H 3800 7350 20  0001 L CNN
+F 2 "" H 3750 7350 60  0000 C CNN
+F 3 "" H 3750 7350 60  0000 C CNN
+	1    3750 7350
+	1    0    0    -1
+$EndComp
+$Comp
+L TESTPOINT TP5
+U 1 1 565A82D6
+P 3750 7450
+F 0 "TP5" H 3750 7400 20  0000 C BNN
+F 1 "TESTPOINT" H 3800 7450 20  0001 L CNN
+F 2 "" H 3750 7450 60  0000 C CNN
+F 3 "" H 3750 7450 60  0000 C CNN
+	1    3750 7450
+	1    0    0    -1
+$EndComp
+$Comp
+L TESTPOINT TP6
+U 1 1 565A833A
+P 3750 7550
+F 0 "TP6" H 3750 7500 20  0000 C BNN
+F 1 "TESTPOINT" H 3800 7550 20  0001 L CNN
+F 2 "" H 3750 7550 60  0000 C CNN
+F 3 "" H 3750 7550 60  0000 C CNN
+	1    3750 7550
+	1    0    0    -1
+$EndComp
+Wire Wire Line
+	3650 6950 4250 6950
+Wire Wire Line
+	3650 7050 4250 7050
+Wire Wire Line
+	3650 7250 4250 7250
+Wire Wire Line
+	3650 7350 4250 7350
+Wire Wire Line
+	3650 7450 4250 7450
+Wire Wire Line
+	3650 7550 4250 7550
+Connection ~ 3750 6950
+Connection ~ 3750 7050
+Connection ~ 3750 7250
+Connection ~ 3750 7350
+Connection ~ 3750 7450
+Connection ~ 3750 7550
 $EndSCHEMATC

Commit message: PCB footprint assignment and floor planning.
Parts:
- C11, C6: footprint (none) -> miniclock:UWX1V470MCL1GB
- TP1, TP2, TP3, TP4, TP5, TP6: footprint (none) -> miniclock:TESTPOINT
Changed lines of the file:
@@
 F 0 "C6" H 2510 4520 50  0000 L CNN
 F 1 "47uF" H 2510 4370 50  0000 L CNN
-F 2 "" H 2500 4450 60  0001 C CNN
+F 2 "miniclock:UWX1V470MCL1GB" H 2500 4450 60  0001 C CNN
 F 3 "" H 2500 4450 60  0000 C CNN
 	1    2500 4450
@@
 F 0 "C11" H 5310 4520 50  0000 L CNN
 F 1 "47uF" H 5310 4370 50  0000 L CNN
-F 2 "" H 5300 4450 60  0001 C CNN
+F 2 "miniclock:UWX1V470MCL1GB" H 5300 4450 60  0001 C CNN
 F 3 "" H 5300 4450 60  0000 C CNN
 	1    5300 4450
@@
 F 0 "TP1" H 3750 6900 20  0000 C BNN
 F 1 "TESTPOINT" H 3800 6950 20  0001 L CNN
-F 2 "" H 3750 6950 60  0000 C CNN
+F 2 "miniclock:TESTPOINT" H 3750 6950 60  0001 C CNN
 F 3 "" H 3750 6950 60  0000 C CNN
 	1    3750 6950
@@
 F 0 "TP2" H 3750 7000 20  0000 C BNN
 F 1 "TESTPOINT" H 3800 7050 20  0001 L CNN
-F 2 "" H 3750 7050 60  0000 C CNN
+F 2 "miniclock:TESTPOINT" H 3750 7050 60  0001 C CNN
 F 3 "" H 3750 7050 60  0000 C CNN
 	1    3750 7050
@@
 F 0 "TP3" H 3750 7200 20  0000 C BNN
 F 1 "TESTPOINT" H 3800 7250 20  0001 L CNN
-F 2 "" H 3750 7250 60  0000 C CNN
+F 2 "miniclock:TESTPOINT" H 3750 7250 60  0001 C CNN
 F 3 "" H 3750 7250 60  0000 C CNN
 	1    3750 7250
@@
 F 0 "TP4" H 3750 7300 20  0000 C BNN
 F 1 "TESTPOINT" H 3800 7350 20  0001 L CNN
-F 2 "" H 3750 7350 60  0000 C CNN
+F 2 "miniclock:TESTPOINT" H 3750 7350 60  0001 C CNN
 F 3 "" H 3750 7350 60  0000 C CNN
 	1    3750 7350
@@
 F 0 "TP5" H 3750 7400 20  0000 C BNN
 F 1 "TESTPOINT" H 3800 7450 20  0001 L CNN
-F 2 "" H 3750 7450 60  0000 C CNN
+F 2 "miniclock:TESTPOINT" H 3750 7450 60  0001 C CNN
 F 3 "" H 3750 7450 60  0000 C CNN
 	1    3750 7450
@@
 F 0 "TP6" H 3750 7500 20  0000 C BNN
 F 1 "TESTPOINT" H 3800 7550 20  0001 L CNN
-F 2 "" H 3750 7550 60  0000 C CNN
+F 2 "miniclock:TESTPOINT" H 3750 7550 60  0001 C CNN
 F 3 "" H 3750 7550 60  0000 C CNN
 	1    3750 7550
